Commit message: commiting all files

File: urdf/obstacles/dynobst.xacro (robot description, xacro)
@@ -11,4 +11,31 @@
     	</plugin>
     </gazebo>
+<!--    <gazebo>-->
+<!--        <plugin name="p3d_base_controller" filename="libgazebo_ros_p3d.so">-->
+<!--            <alwaysOn>true</alwaysOn>-->
+<!--            &lt;!&ndash;<updateRate>50.0</updateRate>&ndash;&gt;-->
+<!--            <bodyName>base_1</bodyName>-->
+<!--            <topicName>odom</topicName>-->
+<!--            <gaussianNoise>0.01</gaussianNoise>-->
+<!--            <frameName>world</frameName>-->
+<!--            <xyzOffsets>0 0 0</xyzOffsets>-->
+<!--            <rpyOffsets>0 0 0</rpyOffsets>-->
+<!--        </plugin>-->
+<!--    </gazebo>-->
+<!--    <gazebo>-->
+<!--        <plugin filename="libgazebo_ros_diff_drive.so" name="differential_drive_controller">-->
+<!--          <alwaysOn>true</alwaysOn>-->
+<!--          <updateRate>20</updateRate>-->
+<!--          <leftJoint>world_base_1</leftJoint>-->
+<!--          <rightJoint>world_base_1</rightJoint>-->
+<!--          <wheelSeparation>0.4</wheelSeparation>-->
+<!--          <wheelDiameter>0.2</wheelDiameter>-->
+<!--          <torque>0.1</torque>-->
+<!--          <commandTopic>cmd_vel</commandTopic>-->
+<!--          <odometryTopic>odom</odometryTopic>-->
+<!--          <odometryFrame>odom</odometryFrame>-->
+<!--          <robotBaseFrame>chassis</robotBaseFrame>-->
+<!--        </plugin>-->
+<!--    </gazebo>-->
 <!--================================================================================================-->
     <link name="world"/>

File: worlds/map.world.xacro (robot description, xacro)
@@ -127,8 +127,8 @@
     </model>
     <state world_name='default'>
-      <sim_time>702 559000000</sim_time>
-      <real_time>618 514921836</real_time>
-      <wall_time>1588012590 562956263</wall_time>
-      <iterations>606535</iterations>
+      <sim_time>792 1000000</sim_time>
+      <real_time>105 759318604</real_time>
+      <wall_time>1588706585 520153731</wall_time>
+      <iterations>89442</iterations>
       <model name='asphalt_plane'>
         <pose frame=''>0 0 0 0 -0 0</pose>
@@ -141,14 +141,4 @@
         </link>
       </model>
-      <model name='cube_20k'>
-        <pose frame=''>5.25802 -4.76127 0.05 2e-06 -2e-06 0.000401</pose>
-        <scale>1 1 1</scale>
-        <link name='link'>
-          <pose frame=''>5.25801 -4.76127 0.55 2e-06 -2e-06 0.000401</pose>
-          <velocity>0 0 0 0 -0 0</velocity>
-          <acceleration>-1.07994 -0.000456 11.799 -3.14071 -0.98169 3.14159</acceleration>
-          <wrench>-1.07994 -0.000456 11.799 0 -0 0</wrench>
-        </link>
-      </model>
       <model name='grey_wall'>
         <pose frame=''>5 -10 0 0 -0 0</pose>
@@ -242,10 +232,10 @@
       </model>
       <model name='wood_cube_2_5cm'>
-        <pose frame=''>3.1622 -4.9867 0.074543 -3.13752 0.000161 0.808678</pose>
-        <scale>1 1 1</scale>
-        <link name='link'>
-          <pose frame=''>3.16216 -4.98667 0.062043 -3.13752 0.000161 0.808678</pose>
-          <velocity>0 0 0 0 -0 0</velocity>
-          <acceleration>0 0 0 4e-06 5e-06 0</acceleration>
+        <pose frame=''>3.16228 -4.98678 0.074181 -3.13327 0.000211 0.808674</pose>
+        <scale>1 1 1</scale>
+        <link name='link'>
+          <pose frame=''>3.1622 -4.98671 0.061681 -3.13327 0.000211 0.808674</pose>
+          <velocity>0 0 0 0 -0 0</velocity>
+          <acceleration>0 0 0 4e-06 6e-06 0</acceleration>
           <wrench>0 0 0 0 -0 0</wrench>
         </link>
@@ -257,5 +247,5 @@
     <gui fullscreen='0'>
       <camera name='user_camera'>
-        <pose frame=''>31.1882 7.11321 34.3746 0 0.749797 3.1162</pose>
+        <pose frame=''>24.458 4.87694 27.8516 0 0.749797 3.1162</pose>
         <view_controller>orbit</view_controller>
         <projection_type>perspective</projection_type>
@@ -684,53 +674,4 @@
       <pose frame=''>3.59557 -5.88146 0 0 -0 0</pose>
     </model>
-    <model name='cube_20k'>
-      <link name='link'>
-        <pose frame=''>0 0 0.5 0 -0 0</pose>
-        <collision name='collision'>
-          <geometry>
-            <mesh>
-              <uri>model://cube_20k/meshes/cube_20k.stl</uri>
-              <scale>1 1 1</scale>
-            </mesh>
-          </geometry>
-          <max_contacts>10</max_contacts>
-          <surface>
-            <contact>
-              <ode/>
-            </contact>
-            <bounce/>
-            <friction>
-              <torsional>
-                <ode/>
-              </torsional>
-              <ode/>
-            </friction>
-          </surface>
-        </collision>
-        <visual name='visual'>
-          <geometry>
-            <mesh>
-              <uri>model://cube_20k/meshes/cube_20k.stl</uri>
-              <scale>1 1 1</scale>
-            </mesh>
-          </geometry>
-        </visual>
-        <self_collide>0</self_collide>
-        <inertial>
-          <inertia>
-            <ixx>1</ixx>
-            <ixy>0</ixy>
-            <ixz>0</ixz>
-            <iyy>1</iyy>
-            <iyz>0</iyz>
-            <izz>1</izz>
-          </inertia>
-          <mass>1</mass>
-        </inertial>
-        <kinematic>0</kinematic>
-        <gravity>1</gravity>
-      </link>
-      <pose frame=''>-0.950673 -1.69493 0 0 -0 0</pose>
-    </model>
   </world>
 </sdf>
